File: ergogen/output/pcbs/corney_island_autorouted.kicad_pcb (KiCad board)
At the start: 2 copper layers, 133.8 x 91.7 mm, 122 parts

Commit message: Update assets
Routing:
- net GND: track 662.5 -> 130.3 mm, vias 31 -> 27
- net VCC: track 634.8 -> 111.0 mm, vias 33 -> 27
- net C0: track 238.7 -> 9.64 mm, vias 2 -> 0
- net C1: track 210.5 -> 9.64 mm, vias 5 -> 0
- net R2: track 203.3 -> 9.63 mm, vias 6 -> 0
- net C3: track 198.5 -> 9.64 mm, vias 4 -> 0
- net C2: track 192.3 -> 9.64 mm, vias 4 -> 0
- net C4: track 181.9 -> 9.64 mm, vias 5 -> 0
- net C5: track 166.5 -> 9.64 mm, vias 4 -> 0
- net R1: track 166.4 -> 9.63 mm, vias 7 -> 0
- net R0: track 165.7 -> 9.63 mm, vias 8 -> 0
- net R3: track 138.5 -> 9.63 mm, vias 4 -> 0
- net ULED_4: track 85.1 -> 13.5 mm, vias 4 -> 2
- net LED_7: track 74.9 -> 13.5 mm, vias 4 -> 2
- net DAT: track 57.0 -> 9.63 mm
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