File: ergogen/output/pcbs/corney_island_wireless_autorouted.kicad_pcb (KiCad board)
At the start: 2 copper layers, 133.8 x 91.7 mm, 96 parts

Commit message: Update assets
Routing:
- net C0: track 218.5 -> 9.64 mm, vias 1 -> 0
- net C3: track 192.8 -> 9.64 mm, vias 5 -> 0
- net C1: track 191.2 -> 9.64 mm, vias 1 -> 0
- net C4: track 187.0 -> 9.64 mm, vias 4 -> 0
- net R0: track 184.0 -> 9.63 mm, vias 9 -> 0
- net R2: track 181.1 -> 9.63 mm, vias 5 -> 0
- net C2: track 179.7 -> 9.64 mm, vias 2 -> 0
- net C5: track 167.5 -> 9.64 mm, vias 2 -> 0
- net R1: track 153.7 -> 9.63 mm, vias 9 -> 0
- net R3: track 126.0 -> 9.63 mm, vias 3 -> 0
- net GND: track 144.8 -> 28.9 mm, vias 2 -> 0
- net RAW: track 57.8 -> 9.64 mm, vias 1 -> 0
- net SDA: track 55.0 -> 9.63 mm, vias 1 -> 0
- net CS: track 53.4 -> 9.63 mm, vias 1 -> 0
- net SCL: track 40.0 -> 9.63 mm, vias 1 -> 0
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